Commit message: still having the same issue, the /odom and wheels frames are not available in Rviz can't find a fix

File: src/warehouse_description/urdf/warehouse_robot.urdf (robot description, URDF)
Before this commit: robot warehouse_robot, 4 links, 3 joints
Links:
- added link base_footprint
- added link imu_link
Joints:
- added joint base_joint: type fixed, parent base_footprint, child base_link, origin xyz=0.0 0.0 0.010 rpy=0 0 0
- added joint imu_joint: type fixed, parent base_link, child imu_link, origin xyz=-0.032 0 0.068 rpy=0 0 0
